File: Transformerless Power Supply.kicad_pcb (KiCad board)
At the start: 2 copper layers, 65.5 x 44.8 mm, 18 parts, among them J1 Screw_Terminal_01x02, J2 Screw_Terminal_01x02, U1 LM7805_TO220

Commit message: PCB with tracks
Parts:
- moved C2 4.07 mm to (162.8, 97.5), turned to -90 degrees
Routing:
- net Net-(D1-K): track 0.00 -> 99.1 mm
- net Net-(D1-A): track 0.00 -> 44.2 mm
- net Net-(J2-Pin_1): track 0.00 -> 26.1 mm
- net Net-(D3-A): track 0.00 -> 24.0 mm
- net Net-(D5-A): track 0.00 -> 18.1 mm
- net Net-(J1-Pin_2): track 0.00 -> 16.6 mm
- net Net-(D6-A): track 0.00 -> 15.8 mm
- net Net-(D7-A): track 0.00 -> 6.18 mm
Other:
- outline, holes or cut-outs redrawn

Commit message: PCB with routing and filled zones
Routing:
- added copper zone on B.Cu, net GND
- added copper zone on F.Cu, net GND
Changed lines of the file:
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@@
 		(net 9)
+	)
+	(zone
+		(net 2)
+		(net_name "GND")
+		(layers "F.Cu" "B.Cu")
+		(hatch edge 0.5)
+		(connect_pads
+			(clearance 0.5)
+		)
+		(min_thickness 0.25)
+		(filled_areas_thickness no)
+		(fill yes
+			(thermal_gap 0.5)
+			(thermal_bridge_width 0.5)
+		)
+		(polygon
+			(pts
+				(xy 124.25 74.5) (xy 190.75 74.5) (xy 190.75 120.25) (xy 124.25 120.25)
+			)
+		)
 	)
 	(embedded_fonts no)
